File: kicad-t6/eeprom.kicad_pcb (KiCad board)
At the start: 2 copper layers, 36 x 20.3 mm, 17 parts, among them J1 PMOD_01x06, J2 PMOD_01x06, SW1 SW_DIP_x04, U1 M24M01-R

Commit message: KiCad v7 upgrade, manual workflow trigger
Other:
- net class 0.25 SMD removed
- net class Default removed
